Commit message: feat: implement forward & inverse dynamics with 3D RViz2 markers and GUI dashboard

File: src/denso_vs6556/urdf/denso_vs6556.urdf (robot description, URDF)
Before this commit: robot denso_vs6556, 7 links, 6 joints
Links:
- link base_link: mass None -> 8.0
- link link_1: mass None -> 4.5
- link link_2: mass None -> 4.2
- link link_3: mass None -> 3.1
- link link_4: mass None -> 2.0
- link link_5: mass None -> 1.2

Commit message: fix(urdf): align Link 4 and kinematic chain to real robot 0-degree candlestick pose

File: src/denso_vs6556/urdf/denso_vs6556.urdf (robot description, URDF)
Before this commit: robot denso_vs6556, 7 links, 6 joints
Joints:
- joint joint_3: origin xyz=0 0.0055 0.270 rpy=0 0 0 -> xyz=0 0.0055 0.270 rpy=0 1.5707963 0
- joint joint_4: origin xyz=-0.088 0.049 0.090 rpy=0 0 0 -> xyz=-0.088 0.049 0.090 rpy=3.1415926 0 0
- joint joint_5: origin xyz=-0.207 0 0 rpy=0 0 0 -> xyz=-0.207 0 0 rpy=3.1415926 0 0
